File: hardware/nibbletronic_KICAD.kicad_pcb (KiCad board)
At the start: 2 copper layers, 259.1 x 29.2 mm, 16 parts, among them P1 DIN_5, SW1 SWITCH_INV, SW2 SWITCH_INV, SW3 SWITCH_INV, SW4 SWITCH_INV, SW5 SWITCH_INV, SW6 SW_PUSH, U1 Arduino_micro, U2 MPX5010DP, U3 Joystick

Commit message: Changed PCBlayout, added new footprints, changed spacing, switched to SMD diode, resistors, buttons and switches.
Parts:
- added D1: D, Diodes_SMD:D_0805, F.Cu at (141.0, 146.1)
- added SW7: Switch_SPDT_x2, Buttons_Switches_SMD:SW_SPDT_PCM12, F.Cu at (254.0, 141.0)
- R1, R2: footprint Resistors_ThroughHole:Resistor_Horizontal_RM10mm -> Resistors_SMD:R_0805_HandSoldering
- SW5: footprint CustomParts:YSS_1203 -> Buttons_Switches_SMD:SW_SPDT_PCM12
- SW6: footprint Buttons_Switches_ThroughHole:SW_PUSH_SMALL -> Buttons_Switches_SMD:SW_SPST_B3S-1000
- moved R1 113.0 mm to (374.6, 123.2), turned to 90 degrees
- moved R2 52.1 mm to (375.9, 146.1)
- moved SW1 15.2 mm to (203.2, 133.3)
- moved RV1 15.2 mm to (335.3, 141.0)
- moved SW2 11.4 mm to (222.2, 133.3)
- moved RV2 11.4 mm to (335.3, 125.7)
- moved SW3 6.35 mm to (242.6, 133.3)
- moved SW5 2.84 mm to (195.6, 123.2), turned to 0 degrees
Connections:
- P1 pad 1: Net-(P1-Pad1) -> (no net)
- P1 pad 3: Net-(P1-Pad3) -> (no net)
- SW6 pad 1: Net-(SW6-Pad1) -> Net-(D1-Pad1)
- SW6 pad 2: /5V -> /REF
- U1 pad 1: Net-(U1-Pad1) -> (no net)
- U1 pad 10: Net-(U1-Pad10) -> (no net)
- U1 pad 11: Net-(U1-Pad11) -> (no net)
- U1 pad 13: Net-(U1-Pad13) -> (no net)
- U1 pad 15: Net-(BT1-Pad1) -> Net-(SW7-Pad2)
- U1 pad 16: Net-(U1-Pad16) -> (no net)
- U1 pad 17: Net-(U1-Pad17) -> (no net)
- U1 pad 18: Net-(U1-Pad18) -> (no net)
- U1 pad 19: Net-(U1-Pad19) -> (no net)
- U1 pad 2: Net-(U1-Pad2) -> (no net)
- U1 pad 22: Net-(U1-Pad22) -> (no net)
- U1 pad 29: Net-(U1-Pad29) -> (no net)
- U1 pad 31: Net-(U1-Pad31) -> (no net)
- U1 pad 32: Net-(U1-Pad32) -> (no net)
- U1 pad 33: Net-(U1-Pad33) -> (no net)
- U1 pad 34: Net-(U1-Pad34) -> (no net)
- U1 pad 4: Net-(SW6-Pad1) -> Net-(D1-Pad1)
- U1 pad 8: Net-(U1-Pad8) -> (no net)
- U1 pad 9: Net-(U1-Pad9) -> (no net)
- U2 pad 1: Net-(SW6-Pad1) -> Net-(D1-Pad2)
- U2 pad 4: Net-(U2-Pad4) -> (no net)
- U2 pad 5: Net-(U2-Pad5) -> (no net)
- U2 pad 6: Net-(U2-Pad6) -> (no net)
Routing:
- net Net-(R1-Pad2): track 73.2 -> 197.5 mm
- net Net-(P1-Pad5): track 133.8 -> 18.2 mm
- net Net-(SW7-Pad2): track 0.00 -> 78.8 mm, vias 0 -> 2
- net Net-(BT1-Pad1): track 129.6 -> 51.4 mm, vias 0 -> 3
- net /5V: track 198.6 -> 265.1 mm, vias 0 -> 4
- net Net-(P1-Pad4): track 76.6 -> 29.2 mm
- net Net-(SW6-Pad1): track 20.6 -> 0.00 mm
- net Net-(D1-Pad1): track 0.00 -> 15.7 mm, vias 0 -> 1
- net Net-(SW1-Pad2): track 45.3 -> 34.5 mm
- net Net-(SW2-Pad2): track 69.6 -> 59.7 mm, vias 0 -> 2
- net Net-(RV1-Pad2): track 146.1 -> 155.5 mm, vias 0 -> 2
- net Net-(RV2-Pad2): track 158.4 -> 153.6 mm, vias 1 -> 3
- net Net-(D1-Pad2): track 0.00 -> 3.90 mm
- net Net-(U1-Pad6): track 126.1 -> 129.2 mm
- net Net-(SW3-Pad2): track 86.7 -> 89.8 mm, vias 1 -> 3
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
Commit message: Changed switches and button due to parts availability, updated BOM
Parts:
- SW5: footprint Buttons_Switches_SMD:SW_SPDT_PCM12 -> CustomParts:ESP40XX
- SW6: footprint Buttons_Switches_SMD:SW_SPST_B3S-1000 -> CustomParts:SMD_Pushbutton_11-22
- SW7: footprint Buttons_Switches_SMD:SW_SPDT_PCM12 -> CustomParts:ESP40XX; moved to B.Cu
- moved SW7 66.1 mm to (320.0, 144.8)
- moved SW4 2.54 mm to (261.6, 133.3)
- moved R2 1.80 mm to (377.2, 144.8), turned to 270 degrees
- moved SW5 1.27 mm to (195.6, 124.5), turned to 180 degrees
Connections:
- P1 pad 1: (no net) -> Net-(P1-Pad1)
- P1 pad 3: (no net) -> Net-(P1-Pad3)
- SW7 pad 1: (no net) -> Net-(SW7-Pad1)
- U1 pad 1: (no net) -> Net-(U1-Pad1)
- U1 pad 10: (no net) -> Net-(U1-Pad10)
- U1 pad 11: (no net) -> Net-(U1-Pad11)
- U1 pad 13: (no net) -> Net-(U1-Pad13)
- U1 pad 16: (no net) -> Net-(U1-Pad16)
- U1 pad 17: (no net) -> Net-(U1-Pad17)
- U1 pad 18: (no net) -> Net-(U1-Pad18)
- U1 pad 19: (no net) -> Net-(U1-Pad19)
- U1 pad 2: (no net) -> Net-(U1-Pad2)
- U1 pad 22: (no net) -> Net-(U1-Pad22)
- U1 pad 29: (no net) -> Net-(U1-Pad29)
- U1 pad 31: (no net) -> Net-(U1-Pad31)
- U1 pad 32: (no net) -> Net-(U1-Pad32)
- U1 pad 33: (no net) -> Net-(U1-Pad33)
- U1 pad 34: (no net) -> Net-(U1-Pad34)
- U1 pad 8: (no net) -> Net-(U1-Pad8)
- U1 pad 9: (no net) -> Net-(U1-Pad9)
- U2 pad 4: (no net) -> Net-(U2-Pad4)
- U2 pad 5: (no net) -> Net-(U2-Pad5)
- U2 pad 6: (no net) -> Net-(U2-Pad6)
Routing:
- net Net-(SW7-Pad2): track 78.8 -> 143.5 mm, vias 2 -> 1
- net Net-(BT1-Pad1): track 51.4 -> 22.9 mm, vias 3 -> 0
- net Net-(SW1-Pad1): track 88.1 -> 77.5 mm, vias 0 -> 2
- net GND: track 0.00 -> 7.62 mm
- net /REF: track 2.83 -> 0.36 mm
- net Net-(SW1-Pad3): track 74.5 -> 76.3 mm
- net Net-(SW4-Pad2): track 101.6 -> 99.9 mm, vias 3 -> 2
- net /5V: track 265.1 -> 263.6 mm
