File: hardware/nibbletronic_KICAD.kicad_pcb (KiCad board)
At the start: 2 copper layers, 31 parts, among them P1 CONN_01X02, P2 CONN_01X09, P3 DIN_5, SW1 Rotary_Encoder_Switch, SW2 Switch_SPDT_x2, SW3 SW_PUSH, U1 Pad, U10 MPX5010DP, U2 Pad, U3 Pad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

Commit message: Hardware 2.0: Touch Buttons and a RotEnc
- Microswitches are replaced by touch sensors with a dedicated IC
- Octave slider has been replaced by two touch sensors
- Added a Rotenc at pins D10-12 and D9 for the Button.
- I2C and all remaining pins (A1, D4, D5, D8, D13), as well as GND, Ref,
3.3/5V have been broken out for easier access
Parts:
- moved R11 10.9 mm to (256.5, 12.7)
- moved R10 10.2 mm to (266.7, 39.4)
Changed lines of the file:
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@@
   )
   (module Resistors_SMD:R_0805_HandSoldering (layer F.Cu)
-    (at 257.81 44.45 180)
+    (at 266.7 39.37 180)
     (descr "Resistor SMD 0805, hand soldering")
     (tags "resistor 0805")
@@
   )
   (module Resistors_SMD:R_0805_HandSoldering (layer F.Cu)
-    (at 247.65 6.35)
+    (at 256.54 12.7)
     (descr "Resistor SMD 0805, hand soldering")
     (tags "resistor 0805")
